Commit message: Use pymeshlab get_geometric_measures() instead of topo.mlx
The result seems about the same.

https://pymeshlab.readthedocs.io/en/latest/filter_list.html#get_geometric_measures

File: robot.urdf (robot description, URDF)
Before this commit: robot pointone, 2 links, 1 joints
Links:
- link bit1: mass 0.01 -> 0.010000; geometry collision mesh filename=bit1.stl; visual mesh filename=bit1.stl
- link bitb: mass 0.01 -> 0.010000; geometry collision mesh filename=bitb.stl; visual mesh filename=bitb.stl
